Commit message: second commit

File: src/dual_arm_control/description/simulation/dummy2/dummy2.urdf (robot description, URDF)
Before this commit: robot dummy2-gripperv2, 11 links, 10 joints
Links:
- removed link camera_1
- removed link camera_eye_1
- removed link figer1_1
- removed link figer2_1
- removed link link1_1
- removed link link2_1
- removed link link3_1
- removed link link4_1
- removed link link5_1
- removed link link6_1
- added link left_base_link, mass 1.2152141810431654; collision mesh filename=package://dual_arm_control/description/simulation/dummy2/me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 scale=0.001 0.001 0.001; visual mesh filename=package://dual_arm_control/description/simulation/dummy2/me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 scale=0.001 0.001 0.001
- added link left_figer1_1, mass 0.0422978780886348; collision mesh filename=package://dual_arm_control/description/simulation/dummy2/me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 scale=0.001 0.001 0.001; visual mesh filename=package://dual_arm_control/description/simulation/dummy2/me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 scale=0.001 0.001 0.001
- added link left_figer2_1, mass 0.042297878145578977; collision mesh filename=package://dual_arm_control/description/simulation/dummy2/me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 scale=0.001 0.001 0.001; visual mesh filename=package://dual_arm_control/description/simulation/dummy2/me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 scale=0.001 0.001 0.001
- added link left_link1_1, mass 0.1444690972471256; collision mesh filename=package://dual_arm_control/description/simulation/dummy2/me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 scale=0.001 0.001 0.001; visual mesh filename=package://dual_arm_control/description/simulation/dummy2/me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 scale=0.001 0.001 0.001
- added link left_link2_1, mass 0.6521077215074461; collision mesh filename=package://dual_arm_control/description/simulation/dummy2/me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 scale=0.001 0.001 0.001; visual mesh filename=package://dual_arm_control/description/simulation/dummy2/me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 scale=0.001 0.001 0.001
- added link left_link3_1, mass 0.9005346433244714; collision mesh filename=package://dual_arm_control/description/simulation/dummy2/me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 scale=0.001 0.001 0.001; visual mesh filename=package://dual_arm_control/description/simulation/dummy2/me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 scale=0.001 0.001 0.001
- added link left_link4_1, mass 0.3580312221089852; collision mesh filename=package://dual_arm_control/description/simulation/dummy2/me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 scale=0.001 0.001 0.001; visual mesh filename=package://dual_arm_control/description/simulation/dummy2/me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 scale=0.001 0.001 0.001
- added link left_link5_1, mass 0.7858738652766984; collision mesh filename=package://dual_arm_control/description/simulation/dummy2/me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 scale=0.001 0.001 0.001; visual mesh filename=package://dual_arm_control/description/simulation/dummy2/me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 scale=0.001 0.001 0.001
- added link left_link6_1, mass 0.604072405055537; collision mesh filename=package://dual_arm_control/description/simulation/dummy2/me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 scale=0.001 0.001 0.001; visual mesh filename=package://dual_arm_control/description/simulation/dummy2/me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 scale=0.001 0.001 0.001
- added link right_base_link, mass 1.2152141810431654; collision mesh filename=package://dual_arm_control/description/simulation/dummy2/me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 scale=0.001 0.001 0.001; visual mesh filename=package://dual_arm_control/description/simulation/dummy2/me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 scale=0.001 0.001 0.001
- added link right_figer1_1, mass 0.0422978780886348; collision mesh filename=package://dual_arm_control/description/simulation/dummy2/me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 scale=0.001 0.001 0.001; visual mesh filename=package://dual_arm_control/description/simulation/dummy2/me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 scale=0.001 0.001 0.001
- added link right_figer2_1, mass 0.042297878145578977; collision mesh filename=package://dual_arm_control/description/simulation/dummy2/me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 scale=0.001 0.001 0.001; visual mesh filename=package://dual_arm_control/description/simulation/dummy2/me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 scale=0.001 0.001 0.001
- added link right_link1_1, mass 0.1444690972471256; collision mesh filename=package://dual_arm_control/description/simulation/dummy2/me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 scale=0.001 0.001 0.001; visual mesh filename=package://dual_arm_control/description/simulation/dummy2/me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 scale=0.001 0.001 0.001
- added link right_link2_1, mass 0.6521077215074461; collision mesh filename=package://dual_arm_control/description/simulation/dummy2/me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 scale=0.001 0.001 0.001; visual mesh filename=package://dual_arm_control/description/simulation/dummy2/me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 scale=0.001 0.001 0.001
- added link right_link3_1, mass 0.9005346433244714; collision mesh filename=package://dual_arm_control/description/simulation/dummy2/me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 scale=0.001 0.001 0.001; visual mesh filename=package://dual_arm_control/description/simulation/dummy2/me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 scale=0.001 0.001 0.001
- added link right_link4_1, mass 0.3580312221089852; collision mesh filename=package://dual_arm_control/description/simulation/dummy2/me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 scale=0.001 0.001 0.001; visual mesh filename=package://dual_arm_control/description/simulation/dummy2/me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 scale=0.001 0.001 0.001
- added link right_link5_1, mass 0.7858738652766984; collision mesh filename=package://dual_arm_control/description/simulation/dummy2/me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 scale=0.001 0.001 0.001; visual mesh filename=package://dual_arm_control/description/simulation/dummy2/me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 scale=0.001 0.001 0.001
- added link right_link6_1, mass 0.604072405055537; collision mesh filename=package://dual_arm_control/description/simulation/dummy2/me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 scale=0.001 0.001 0.001; visual mesh filename=package://dual_arm_control/description/simulation/dummy2/me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 scale=0.001 0.001 0.001
- link base_link: mass 1.2152141810431654 -> 2.0; geometry collision box size=0.4 0.2 0.1; visual box size=0.6 0.2 0.1
Joints:
- removed joint camera
- removed joint camera_eye
- removed joint figer1
- removed joint figer2
- removed joint joint1
- removed joint joint2
- removed joint joint3
- removed joint joint4
- removed joint joint5
- removed joint joint6
- added joint left_base_joint: type fixed, parent base_link, child left_base_link, origin xyz=0.2 0 0.05 rpy=0 0 0
- added joint left_figer1: type prismatic, parent left_link6_1, child left_figer1_1, origin xyz=0.012824 0.074462 -0.0001 rpy=0 0 0, axis 1.0 -0.0 0.0, limit lower=0.0 upper=0.028 effort=100 velocity=100
- added joint left_figer2: type prismatic, parent left_link6_1, child left_figer2_1, origin xyz=-0.012176 0.074462 0.0 rpy=0 0 0, axis 1.0 -0.0 0.0, limit lower=-0.028 upper=0.0 effort=100 velocity=100
- added joint left_joint1: type revolute, parent left_base_link, child left_link1_1, origin xyz=0.0 0.0 0.096 rpy=0 0 0, axis 0.0 -0.0 -1.0, limit lower=-3.001966 upper=3.001966 effort=100 velocity=100
- added joint left_joint2: type revolute, parent left_link1_1, child left_link2_1, origin xyz=-0.011639 0.034477 0.0285 rpy=0 0 0, axis 1.0 0.0 -0.0, limit lower=-1.570796 upper=1.308997 effort=100 velocity=100
- added joint left_joint3: type revolute, parent left_link2_1, child left_link3_1, origin xyz=0.03615 0.0 0.168 rpy=0 0 0, axis -1.0 -0.0 -0.0, limit lower=-1.500983 upper=1.570796 effort=100 velocity=100
- added joint left_joint4: type revolute, parent left_link3_1, child left_link4_1, origin xyz=-0.013162 0.0041 0.062467 rpy=0 0 0, axis 0.0 -1.0 0.0, limit lower=-3.141593 upper=3.141593 effort=100 velocity=100
- added joint left_joint5: type revolute, parent left_link4_1, child left_link5_1, origin xyz=0.0213 0.11 0.0 rpy=0 0 0, axis -1.0 -0.0 -0.0, limit lower=-1.919862 upper=2.094395 effort=100 velocity=100
- added joint left_joint6: type revolute, parent left_link5_1, child left_link6_1, origin xyz=-0.019822 0.1195 -0.001226 rpy=0 0 0, axis 0.0 -1.0 -0.0, limit lower=-3.141593 upper=3.141593 effort=100 velocity=100
- added joint right_base_joint: type fixed, parent base_link, child right_base_link, origin xyz=-0.2 0 0.05 rpy=0 0 0
- added joint right_figer1: type prismatic, parent right_link6_1, child right_figer1_1, origin xyz=0.012824 0.074462 -0.0001 rpy=0 0 0, axis 1.0 -0.0 0.0, limit lower=0.0 upper=0.028 effort=100 velocity=100
- added joint right_figer2: type prismatic, parent right_link6_1, child right_figer2_1, origin xyz=-0.012176 0.074462 0.0 rpy=0 0 0, axis 1.0 -0.0 0.0, limit lower=-0.028 upper=0.0 effort=100 velocity=100
- added joint right_joint1: type revolute, parent right_base_link, child right_link1_1, origin xyz=0.0 0.0 0.096 rpy=0 0 0, axis 0.0 -0.0 -1.0, limit lower=-3.001966 upper=3.001966 effort=100 velocity=100
- added joint right_joint2: type revolute, parent right_link1_1, child right_link2_1, origin xyz=-0.011639 0.034477 0.0285 rpy=0 0 0, axis 1.0 0.0 -0.0, limit lower=-1.570796 upper=1.308997 effort=100 velocity=100
- added joint right_joint3: type revolute, parent right_link2_1, child right_link3_1, origin xyz=0.03615 0.0 0.168 rpy=0 0 0, axis -1.0 -0.0 -0.0, limit lower=-1.500983 upper=1.570796 effort=100 velocity=100
- added joint right_joint4: type revolute, parent right_link3_1, child right_link4_1, origin xyz=-0.013162 0.0041 0.062467 rpy=0 0 0, axis 0.0 -1.0 0.0, limit lower=-3.141593 upper=3.141593 effort=100 velocity=100
- added joint right_joint5: type revolute, parent right_link4_1, child right_link5_1, origin xyz=0.0213 0.11 0.0 rpy=0 0 0, axis -1.0 -0.0 -0.0, limit lower=-1.919862 upper=2.094395 effort=100 velocity=100
- added joint right_joint6: type revolute, parent right_link5_1, child right_link6_1, origin xyz=-0.019822 0.1195 -0.001226 rpy=0 0 0, axis 0.0 -1.0 -0.0, limit lower=-3.141593 upper=3.141593 effort=100 velocity=100
